File: cv-gate.kicad_sch (KiCad schematic)
At the start: 49 parts, among them J1 Conn_01x06_Socket, J2 Conn_01x06_Socket, J3 Conn_02x05_Odd_Even, U2 TL074, U3 TL074, U4 MCP1703Ax-500xxDB

Commit message: Moved I/O buffering to interface board, add license
Parts:
- removed C15: 100pF, Capacitor_SMD:C_0805_2012Metric_Pad1.18x1.45mm_HandSolder, symbol Device:C
- added R4: 10K, Resistor_SMD:R_0805_2012Metric_Pad1.20x1.40mm_HandSolder, symbol Device:R_US
- R13, R15: value 100K -> 1K
Connections:
- net CV_IN_BUFFERED: now also J2.2 (Pin_2); no longer U3.1, U3.2 (-)
- net GND: now also U3.3 (+)
- net THRESHOLD_NEGATIVE: now also U3.1, R4.1; no longer J2.5 (Pin_5)
- net THRESHOLD_POSITIVE: now also U3.2 (-), R4.2
- removed net CV_IN_RAW: J2.2 (Pin_2), U3.3 (+)
- net CV_OUT_BUFFERED renamed CV_OUT_RAW
Other:
- note added: "Threshold Inverter"
- note removed: "CV Input"
- note removed: "CV_IN_RAW has 1K series R on interface board"
- moved on the sheet: J1

Commit message: Add bom, 3d model
Parts:
- C12, C8: value 1uF -> 0.1uF
- U1: value ~ -> TMUX6121
Other:
- moved on the sheet: C12, C8
